Commit message: add reaction wheel and wall environment

File: robots/a1_description/xacro/leg.xacro (robot description, xacro)
@@ -149,4 +149,12 @@
                     <sphere radius="${foot_radius}"/>
                 </geometry>
+	                <surface>
+                 <friction>
+                  <ode>
+                        <mu>1.0</mu>
+                        <mu2>1.0</mu2>
+                  </ode>
+                 </friction>
+                </surface>
             </collision>
             <inertial>

File: robots/a1_description/xacro/robot.xacro (robot description, xacro)
@@ -42,5 +42,5 @@
             <origin rpy="0 0 0" xyz="0 0 0"/>
             <geometry>
-                <box size="${trunk_length} ${trunk_width} ${trunk_height}"/>
+                <mesh filename="package://a1_description/meshes/trunk.dae" scale="1 1 1"/>
             </geometry>
         </collision>
