Commit message: can move one step  but very unstable

File: robots/a1_description/xacro/const.xacro (robot description, xacro)
@@ -29,6 +29,6 @@
     <xacro:property name="hip_offset" value="0.065"/>
     <!-- joint limits -->
-    <xacro:property name="damping" value="0"/>
-    <xacro:property name="friction" value="0"/>
+    <xacro:property name="damping" value="1e-3"/>
+    <xacro:property name="friction" value="1e-3"/>
     <xacro:property name="hip_max" value="46"/>
     <xacro:property name="hip_min" value="-46"/>

Commit message: updated A1 trunk mass parameters

File: robots/a1_description/xacro/const.xacro (robot description, xacro)
@@ -45,14 +45,14 @@
     <!-- dynamics inertial value -->
     <!-- trunk -->
-    <xacro:property name="trunk_mass" value="4.713"/>
-    <xacro:property name="trunk_com_x" value="0.012731"/>
-    <xacro:property name="trunk_com_y" value="0.002186"/>
-    <xacro:property name="trunk_com_z" value="0.000515"/>
-    <xacro:property name="trunk_ixx" value="0.016839930"/>
-    <xacro:property name="trunk_ixy" value="0.000083902"/>
-    <xacro:property name="trunk_ixz" value="0.000597679"/>
-    <xacro:property name="trunk_iyy" value="0.056579028"/>
-    <xacro:property name="trunk_iyz" value="0.000025134"/>
-    <xacro:property name="trunk_izz" value="0.064713601"/>
+    <xacro:property name="trunk_mass" value="6.0"/>
+    <xacro:property name="trunk_com_x" value="0.0000"/>
+    <xacro:property name="trunk_com_y" value="0.0041"/>
+    <xacro:property name="trunk_com_z" value="-0.0005"/>
+    <xacro:property name="trunk_ixx" value="0.0158533"/>
+    <xacro:property name="trunk_ixy" value="-0.0000366"/>
+    <xacro:property name="trunk_ixz" value="-0.0000611"/>
+    <xacro:property name="trunk_iyy" value="0.0377999"/>
+    <xacro:property name="trunk_iyz" value="-0.0000275"/>
+    <xacro:property name="trunk_izz" value="0.0456542"/>
     <!-- hip (left front) -->
     <xacro:property name="hip_mass" value="0.696"/>

Commit message: improve sim

File: robots/a1_description/xacro/const.xacro (robot description, xacro)
@@ -29,6 +29,6 @@
     <xacro:property name="hip_offset" value="0.065"/>
     <!-- joint limits -->
-    <xacro:property name="damping" value="1e-3"/>
-    <xacro:property name="friction" value="1e-3"/>
+    <xacro:property name="damping" value="1e-2"/>
+    <xacro:property name="friction" value="1e-2"/>
     <xacro:property name="hip_max" value="46"/>
     <xacro:property name="hip_min" value="-46"/>

File: robots/a1_description/xacro/gazebo.xacro (robot description, xacro)
@@ -20,6 +20,17 @@
         </plugin>
     </gazebo>
+    <gazebo>
+        <plugin name="p3d" filename="libgazebo_ros_p3d.so">
+            <always_on>true</always_on>
+            <update_rate>200</update_rate>
+            <bodyName>base</bodyName>
+            <topicName>/torso_odom</topicName>
+            <frameName>world</frameName>
+            <xyzOffset>0 0 0</xyzOffset>
+            <rpyOffset>0 0 0</rpyOffset>
+        </plugin>
+    </gazebo>
     <!-- Show the trajectory of trunk center. -->
-    <!-- <gazebo>
+    <gazebo>
         <plugin name="3dplot" filename="libLinkPlot3DPlugin.so">
             <frequency>10</frequency>
@@ -30,7 +41,7 @@
             </plot>
         </plugin>
-    </gazebo> -->
+    </gazebo>
     <!-- Show the trajectory of foot. You can add another trajectory about another foot. -->
-    <!-- <gazebo>
+    <gazebo>
         <plugin name="3dplot" filename="libLinkPlot3DPlugin.so">
             <frequency>100</frequency>
@@ -41,5 +52,5 @@
             </plot>
         </plugin>
-    </gazebo> -->
+    </gazebo>
     <gazebo>
         <plugin filename="libgazebo_ros_force.so" name="gazebo_ros_force">
@@ -52,5 +63,5 @@
         <sensor name="imu_sensor" type="imu">
             <always_on>true</always_on>
-            <update_rate>100</update_rate>
+            <update_rate>400</update_rate>
             <visualize>true</visualize>
             <topic>__default_topic__</topic>
@@ -58,5 +69,5 @@
                 <topicName>trunk_imu</topicName>
                 <bodyName>imu_link</bodyName>
-                <updateRateHZ>200.0</updateRateHZ>
+                <updateRateHZ>400.0</updateRateHZ>
                 <gaussianNoise>0.0</gaussianNoise>
                 <xyzOffset>0 0 0</xyzOffset>

Commit message: increase model damping

File: robots/a1_description/xacro/const.xacro (robot description, xacro)
@@ -29,5 +29,5 @@
     <xacro:property name="hip_offset" value="0.065"/>
     <!-- joint limits -->
-    <xacro:property name="damping" value="1e-2"/>
+    <xacro:property name="damping" value="1e-1"/>
     <xacro:property name="friction" value="1e-2"/>
     <xacro:property name="hip_max" value="46"/>

File: robots/a1_description/xacro/gazebo.xacro (robot description, xacro)
@@ -33,25 +33,4 @@
     <!-- Show the trajectory of trunk center. -->
     <gazebo>
-        <plugin name="3dplot" filename="libLinkPlot3DPlugin.so">
-            <frequency>10</frequency>
-            <plot>
-                <link>base</link>
-                <pose>0 0 0 0 0 0</pose>
-                <material>Gazebo/Yellow</material>
-            </plot>
-        </plugin>
-    </gazebo>
-    <!-- Show the trajectory of foot. You can add another trajectory about another foot. -->
-    <gazebo>
-        <plugin name="3dplot" filename="libLinkPlot3DPlugin.so">
-            <frequency>100</frequency>
-            <plot>
-                <link>FL_foot</link>
-                <pose>0 0 0 0 0 0</pose>
-                <material>Gazebo/Green</material>
-            </plot>
-        </plugin>
-    </gazebo>
-    <gazebo>
         <plugin filename="libgazebo_ros_force.so" name="gazebo_ros_force">
             <bodyName>trunk</bodyName>
@@ -63,5 +42,5 @@
         <sensor name="imu_sensor" type="imu">
             <always_on>true</always_on>
-            <update_rate>400</update_rate>
+            <update_rate>200</update_rate>
             <visualize>true</visualize>
             <topic>__default_topic__</topic>
@@ -69,5 +48,5 @@
                 <topicName>trunk_imu</topicName>
                 <bodyName>imu_link</bodyName>
-                <updateRateHZ>400.0</updateRateHZ>
+                <updateRateHZ>200.0</updateRateHZ>
                 <gaussianNoise>0.0</gaussianNoise>
                 <xyzOffset>0 0 0</xyzOffset>

Commit message: update packages

File: robots/a1_description/xacro/const.xacro (robot description, xacro)
@@ -29,6 +29,6 @@
     <xacro:property name="hip_offset" value="0.065"/>
     <!-- joint limits -->
-    <xacro:property name="damping" value="1e-1"/>
-    <xacro:property name="friction" value="1e-2"/>
+    <xacro:property name="damping" value="0"/>
+    <xacro:property name="friction" value="0"/>
     <xacro:property name="hip_max" value="46"/>
     <xacro:property name="hip_min" value="-46"/>
@@ -43,5 +43,5 @@
     <xacro:property name="calf_velocity_max" value="21"/>
     <xacro:property name="calf_torque_max" value="33.5"/>
-    <!-- dynamics inertial value -->
+    <!-- dynamics inertial value        total 13.9kg -->
     <!-- trunk -->
     <xacro:property name="trunk_mass" value="6.0"/>
@@ -56,36 +56,36 @@
     <xacro:property name="trunk_izz" value="0.0456542"/>
     <!-- hip (left front) -->
-    <xacro:property name="hip_mass" value="0.696"/>
-    <xacro:property name="hip_com_x" value="-0.003311"/>
-    <xacro:property name="hip_com_y" value="0.000635"/>
-    <xacro:property name="hip_com_z" value="0.000031"/>
-    <xacro:property name="hip_ixx" value="0.000469246"/>
-    <xacro:property name="hip_ixy" value="-0.000009409"/>
-    <xacro:property name="hip_ixz" value="-0.000000342"/>
-    <xacro:property name="hip_iyy" value="0.000807490"/>
-    <xacro:property name="hip_iyz" value="-0.000000466"/>
-    <xacro:property name="hip_izz" value="0.000552929"/>
+    <xacro:property name="hip_mass" value="0.595"/>
+    <xacro:property name="hip_com_x" value="-0.003875"/>
+    <xacro:property name="hip_com_y" value="0.001622"/>
+    <xacro:property name="hip_com_z" value="0.000042"/>
+    <xacro:property name="hip_ixx" value="0.000402747"/>
+    <xacro:property name="hip_ixy" value="-0.000008709"/>
+    <xacro:property name="hip_ixz" value="-0.000000297"/>
+    <xacro:property name="hip_iyy" value="0.000691123"/>
+    <xacro:property name="hip_iyz" value="-0.000000545"/>
+    <xacro:property name="hip_izz" value="0.000487919"/>
     <!-- thigh -->
-    <xacro:property name="thigh_mass" value="1.013"/>
-    <xacro:property name="thigh_com_x" value="-0.003237"/>
-    <xacro:property name="thigh_com_y" value="-0.022327"/>
-    <xacro:property name="thigh_com_z" value="-0.027326"/>
-    <xacro:property name="thigh_ixx" value="0.005529065"/>
-    <xacro:property name="thigh_ixy" value="0.000004825"/>
-    <xacro:property name="thigh_ixz" value="0.000343869"/>
-    <xacro:property name="thigh_iyy" value="0.005139339"/>
-    <xacro:property name="thigh_iyz" value="0.000022448"/>
-    <xacro:property name="thigh_izz" value="0.001367788"/>
+    <xacro:property name="thigh_mass" value="0.888"/>
+    <xacro:property name="thigh_com_x" value="-0.003574"/>
+    <xacro:property name="thigh_com_y" value="-0.019529"/>
+    <xacro:property name="thigh_com_z" value="-0.030323"/>
+    <xacro:property name="thigh_ixx" value="0.005251806"/>
+    <xacro:property name="thigh_ixy" value="-0.000002168"/>
+    <xacro:property name="thigh_ixz" value="0.000346889"/>
+    <xacro:property name="thigh_iyy" value="0.005000475"/>
+    <xacro:property name="thigh_iyz" value="-0.000028174"/>
+    <xacro:property name="thigh_izz" value="0.001110200"/>
     <!-- calf -->
-    <xacro:property name="calf_mass" value="0.166"/>
-    <xacro:property name="calf_com_x" value="0.006435"/>
-    <xacro:property name="calf_com_y" value="0.0"/>
-    <xacro:property name="calf_com_z" value="-0.107388"/>
-    <xacro:property name="calf_ixx" value="0.002997972"/>
+    <xacro:property name="calf_mass" value="0.151"/>
+    <xacro:property name="calf_com_x" value="0.007105"/>
+    <xacro:property name="calf_com_y" value="-0.000239"/>
+    <xacro:property name="calf_com_z" value="-0.096933"/>
+    <xacro:property name="calf_ixx" value="0.002344758"/>
     <xacro:property name="calf_ixy" value="0.0"/>
-    <xacro:property name="calf_ixz" value="-0.000141163"/>
-    <xacro:property name="calf_iyy" value="0.003014022"/>
+    <xacro:property name="calf_ixz" value="-0.000141275"/>
+    <xacro:property name="calf_iyy" value="0.002360755"/>
     <xacro:property name="calf_iyz" value="0.0"/>
-    <xacro:property name="calf_izz" value="0.000032426"/>
+    <xacro:property name="calf_izz" value="0.000031158"/>
     <!-- foot -->
     <xacro:property name="foot_mass" value="0.06"/>

File: robots/a1_description/xacro/gazebo.xacro (robot description, xacro)
@@ -8,27 +8,26 @@
         </plugin>
     </gazebo>
-    <!-- simulate a body pose sensor -->
+    <!-- Show the trajectory of trunk center. -->
     <gazebo>
-        <plugin name="p3d" filename="libgazebo_ros_p3d.so">
-        <alwaysOn>true</alwaysOn>
-        <updateRate>100.0</updateRate>
-        <bodyName>base</bodyName>
-        <topicName>body_pose_ground_truth</topicName>
-        <frameName>world</frameName>
-        <xyzOffsets>0 0 0.0</xyzOffsets>
-        <rpyOffsets>0 0 0.0</rpyOffsets>
-        </plugin>
-    </gazebo>
-    <gazebo>
-        <plugin name="p3d" filename="libgazebo_ros_p3d.so">
-            <always_on>true</always_on>
-            <update_rate>200</update_rate>
-            <bodyName>base</bodyName>
-            <topicName>/torso_odom</topicName>
-            <frameName>world</frameName>
-            <xyzOffset>0 0 0</xyzOffset>
-            <rpyOffset>0 0 0</rpyOffset>
-        </plugin>
-    </gazebo>
+        <plugin name="3dplot" filename="libLinkPlot3DPlugin.so">
+            <frequency>10</frequency>
+            <plot>
+                <link>base</link>
+                <pose>0 0 0 0 0 0</pose>
+                <material>Gazebo/Yellow</material>
+            </plot>
+        </plugin>
+    </gazebo>
+    <!-- Show the trajectory of foot. You can add another trajectory about another foot. -->
+    <!-- <gazebo>
+        <plugin name="3dplot" filename="libLinkPlot3DPlugin.so">
+            <frequency>100</frequency>
+            <plot>
+                <link>FL_foot</link>
+                <pose>0 0 0 0 0 0</pose>
+                <material>Gazebo/Green</material>
+            </plot>
+        </plugin>
+    </gazebo> -->
     <gazebo>
         <plugin filename="libgazebo_ros_force.so" name="gazebo_ros_force">
@@ -41,5 +40,5 @@
         <sensor name="imu_sensor" type="imu">
             <always_on>true</always_on>
-            <update_rate>400</update_rate>
+            <update_rate>1000</update_rate>
             <visualize>true</visualize>
             <topic>__default_topic__</topic>
@@ -47,6 +46,6 @@
                 <topicName>trunk_imu</topicName>
                 <bodyName>imu_link</bodyName>
-                <updateRateHZ>400.0</updateRateHZ>
-                <gaussianNoise>0.001</gaussianNoise>
+                <updateRateHZ>1000.0</updateRateHZ>
+                <gaussianNoise>0.0</gaussianNoise>
                 <xyzOffset>0 0 0</xyzOffset>
                 <rpyOffset>0 0 0</rpyOffset>

File: robots/a1_description/xacro/leg.xacro (robot description, xacro)
@@ -149,12 +149,4 @@
                     <sphere radius="${foot_radius}"/>
                 </geometry>
-	                <surface>
-                 <friction>
-                  <ode>
-                        <mu>1.0</mu>
-                        <mu2>1.0</mu2>
-                  </ode>
-                 </friction>
-                </surface>
             </collision>
             <inertial>

File: robots/a1_description/xacro/robot.xacro (robot description, xacro)
@@ -6,4 +6,5 @@
     <xacro:include filename="$(find a1_description)/xacro/stairs.xacro"/>
     <xacro:include filename="$(find a1_description)/xacro/gazebo.xacro"/>
+    <!-- <xacro:include filename="$(find a1_gazebo)/launch/stairs.urdf.xacro"/> -->
     <!-- <xacro:stairs stairs="15" xpos="0" ypos="0" zpos="0" /> -->
     <!-- Rollover Protection mode will add an additional stick on the top, use "true" or "false" to switch it. -->
@@ -42,5 +43,5 @@
             <origin rpy="0 0 0" xyz="0 0 0"/>
             <geometry>
-                <mesh filename="package://a1_description/meshes/trunk.dae" scale="1 1 1"/>
+                <box size="${trunk_length} ${trunk_width} ${trunk_height}"/>
             </geometry>
         </collision>

File: robots/aliengo_description/xacro/const.xacro (robot description, xacro)
@@ -20,9 +20,9 @@
     <xacro:property name="stick_length" value="0.2"/>
     <!-- kinematic value -->
-    <xacro:property name="thigh_offset" value="0.083"/>
+    <xacro:property name="thigh_offset" value="0.0868"/>
     <xacro:property name="thigh_length" value="0.25"/>
     <xacro:property name="calf_length" value="0.25"/>
     <!-- leg offset from trunk center value -->
-    <xacro:property name="leg_offset_x" value="0.2399"/>
+    <xacro:property name="leg_offset_x" value="0.2407"/>
     <xacro:property name="leg_offset_y" value="0.051"/>
     <xacro:property name="trunk_offset_z" value="0.01675"/>
@@ -34,12 +34,14 @@
     <xacro:property name="hip_position_min" value="${-70*PI/180.0}"/>
     <xacro:property name="hip_velocity_max" value="20"/>
-    <xacro:property name="hip_torque_max" value="44"/>
+    <xacro:property name="hip_torque_max" value="35.278"/>
+    <xacro:property name="thigh_position_max" value="${240*PI/180.0}"/>
+    <xacro:property name="thigh_position_min" value="${-120*PI/180.0}"/>
     <xacro:property name="thigh_velocity_max" value="20"/>
-    <xacro:property name="thigh_torque_max" value="44"/>
+    <xacro:property name="thigh_torque_max" value="35.278"/>
     <xacro:property name="calf_position_max" value="${-37*PI/180.0}"/>
     <xacro:property name="calf_position_min" value="${-159*PI/180.0}"/>
-    <xacro:property name="calf_velocity_max" value="16"/>
-    <xacro:property name="calf_torque_max" value="55"/>
-    <!-- dynamics inertial value -->
+    <xacro:property name="calf_velocity_max" value="15.89"/>
+    <xacro:property name="calf_torque_max" value="44.4"/>
+    <!-- dynamics inertial value        total 22.0kg -->
     <!-- trunk -->
     <xacro:property name="trunk_mass" value="11.041"/>

File: robots/go1_description/xacro/gazebo.xacro (robot description, xacro)
@@ -8,27 +8,26 @@
         </plugin>
     </gazebo>
-    <!-- simulate a body pose sensor -->
+    <!-- Show the trajectory of trunk center. -->
     <gazebo>
-        <plugin name="p3d" filename="libgazebo_ros_p3d.so">
-        <alwaysOn>true</alwaysOn>
-        <updateRate>100.0</updateRate>
-        <bodyName>base</bodyName>
-        <topicName>body_pose_ground_truth</topicName>
-        <frameName>world</frameName>
-        <xyzOffsets>0 0 0.0</xyzOffsets>
-        <rpyOffsets>0 0 0.0</rpyOffsets>
-        </plugin>
-    </gazebo>
-    <gazebo>
-        <plugin name="p3d" filename="libgazebo_ros_p3d.so">
-            <always_on>true</always_on>
-            <update_rate>200</update_rate>
-            <bodyName>base</bodyName>
-            <topicName>/torso_odom</topicName>
-            <frameName>world</frameName>
-            <xyzOffset>0 0 0</xyzOffset>
-            <rpyOffset>0 0 0</rpyOffset>
-        </plugin>
-    </gazebo>
+        <plugin name="3dplot" filename="libLinkPlot3DPlugin.so">
+            <frequency>10</frequency>
+            <plot>
+                <link>base</link>
+                <pose>0 0 0 0 0 0</pose>
+                <material>Gazebo/Yellow</material>
+            </plot>
+        </plugin>
+    </gazebo>
+    <!-- Show the trajectory of foot. You can add another trajectory about another foot. -->
+    <!-- <gazebo>
+        <plugin name="3dplot" filename="libLinkPlot3DPlugin.so">
+            <frequency>100</frequency>
+            <plot>
+                <link>FL_foot</link>
+                <pose>0 0 0 0 0 0</pose>
+                <material>Gazebo/Green</material>
+            </plot>
+        </plugin>
+    </gazebo> -->
     <gazebo>
         <plugin filename="libgazebo_ros_force.so" name="gazebo_ros_force">

File: robots/laikago_description/xacro/const.xacro (robot description, xacro)
@@ -33,14 +33,14 @@
     <xacro:property name="hip_max" value="60"/>
     <xacro:property name="hip_min" value="-50"/>
-    <xacro:property name="hip_velocity_max" value="52.4"/>
-    <xacro:property name="hip_torque_max" value="20"/>
+    <xacro:property name="hip_velocity_max" value="27"/>
+    <xacro:property name="hip_torque_max" value="18.954"/>
     <xacro:property name="thigh_max" value="225"/>
     <xacro:property name="thigh_min" value="-30"/>
-    <xacro:property name="thigh_velocity_max" value="28.6"/>
-    <xacro:property name="thigh_torque_max" value="55"/>
+    <xacro:property name="thigh_velocity_max" value="12.794"/>
+    <xacro:property name="thigh_torque_max" value="40"/>
     <xacro:property name="calf_max" value="-35"/>
     <xacro:property name="calf_min" value="-159"/>
-    <xacro:property name="calf_velocity_max" value="28.6"/>
-    <xacro:property name="calf_torque_max" value="55"/>
+    <xacro:property name="calf_velocity_max" value="12.794"/>
+    <xacro:property name="calf_torque_max" value="40"/>
     <!-- dynamics inertial value -->
     <!-- trunk -->
