Commit message: a1_description

File: robots/a1_description/xacro/const.xacro (robot description, xacro)
@@ -29,6 +29,6 @@
     <xacro:property name="hip_offset" value="0.065"/>
     <!-- joint limits -->
-    <xacro:property name="damping" value="0"/>
-    <xacro:property name="friction" value="0"/>
+    <xacro:property name="damping" value="1e-1"/>
+    <xacro:property name="friction" value="1e-2"/>
     <xacro:property name="hip_max" value="46"/>
     <xacro:property name="hip_min" value="-46"/>
@@ -43,5 +43,5 @@
     <xacro:property name="calf_velocity_max" value="21"/>
     <xacro:property name="calf_torque_max" value="33.5"/>
-    <!-- dynamics inertial value        total 13.9kg -->
+    <!-- dynamics inertial value -->
     <!-- trunk -->
     <xacro:property name="trunk_mass" value="6.0"/>
@@ -56,36 +56,36 @@
     <xacro:property name="trunk_izz" value="0.0456542"/>
     <!-- hip (left front) -->
-    <xacro:property name="hip_mass" value="0.595"/>
-    <xacro:property name="hip_com_x" value="-0.003875"/>
-    <xacro:property name="hip_com_y" value="0.001622"/>
-    <xacro:property name="hip_com_z" value="0.000042"/>
-    <xacro:property name="hip_ixx" value="0.000402747"/>
-    <xacro:property name="hip_ixy" value="-0.000008709"/>
-    <xacro:property name="hip_ixz" value="-0.000000297"/>
-    <xacro:property name="hip_iyy" value="0.000691123"/>
-    <xacro:property name="hip_iyz" value="-0.000000545"/>
-    <xacro:property name="hip_izz" value="0.000487919"/>
+    <xacro:property name="hip_mass" value="0.696"/>
+    <xacro:property name="hip_com_x" value="-0.003311"/>
+    <xacro:property name="hip_com_y" value="0.000635"/>
+    <xacro:property name="hip_com_z" value="0.000031"/>
+    <xacro:property name="hip_ixx" value="0.000469246"/>
+    <xacro:property name="hip_ixy" value="-0.000009409"/>
+    <xacro:property name="hip_ixz" value="-0.000000342"/>
+    <xacro:property name="hip_iyy" value="0.000807490"/>
+    <xacro:property name="hip_iyz" value="-0.000000466"/>
+    <xacro:property name="hip_izz" value="0.000552929"/>
     <!-- thigh -->
-    <xacro:property name="thigh_mass" value="0.888"/>
-    <xacro:property name="thigh_com_x" value="-0.003574"/>
-    <xacro:property name="thigh_com_y" value="-0.019529"/>
-    <xacro:property name="thigh_com_z" value="-0.030323"/>
-    <xacro:property name="thigh_ixx" value="0.005251806"/>
-    <xacro:property name="thigh_ixy" value="-0.000002168"/>
-    <xacro:property name="thigh_ixz" value="0.000346889"/>
-    <xacro:property name="thigh_iyy" value="0.005000475"/>
-    <xacro:property name="thigh_iyz" value="-0.000028174"/>
-    <xacro:property name="thigh_izz" value="0.001110200"/>
+    <xacro:property name="thigh_mass" value="1.013"/>
+    <xacro:property name="thigh_com_x" value="-0.003237"/>
+    <xacro:property name="thigh_com_y" value="-0.022327"/>
+    <xacro:property name="thigh_com_z" value="-0.027326"/>
+    <xacro:property name="thigh_ixx" value="0.005529065"/>
+    <xacro:property name="thigh_ixy" value="0.000004825"/>
+    <xacro:property name="thigh_ixz" value="0.000343869"/>
+    <xacro:property name="thigh_iyy" value="0.005139339"/>
+    <xacro:property name="thigh_iyz" value="0.000022448"/>
+    <xacro:property name="thigh_izz" value="0.001367788"/>
     <!-- calf -->
-    <xacro:property name="calf_mass" value="0.151"/>
-    <xacro:property name="calf_com_x" value="0.007105"/>
-    <xacro:property name="calf_com_y" value="-0.000239"/>
-    <xacro:property name="calf_com_z" value="-0.096933"/>
-    <xacro:property name="calf_ixx" value="0.002344758"/>
+    <xacro:property name="calf_mass" value="0.166"/>
+    <xacro:property name="calf_com_x" value="0.006435"/>
+    <xacro:property name="calf_com_y" value="0.0"/>
+    <xacro:property name="calf_com_z" value="-0.107388"/>
+    <xacro:property name="calf_ixx" value="0.002997972"/>
     <xacro:property name="calf_ixy" value="0.0"/>
-    <xacro:property name="calf_ixz" value="-0.000141275"/>
-    <xacro:property name="calf_iyy" value="0.002360755"/>
+    <xacro:property name="calf_ixz" value="-0.000141163"/>
+    <xacro:property name="calf_iyy" value="0.003014022"/>
     <xacro:property name="calf_iyz" value="0.0"/>
-    <xacro:property name="calf_izz" value="0.000031158"/>
+    <xacro:property name="calf_izz" value="0.000032426"/>
     <!-- foot -->
     <xacro:property name="foot_mass" value="0.06"/>

File: robots/a1_description/xacro/gazebo.xacro (robot description, xacro)
@@ -8,26 +8,28 @@
         </plugin>
     </gazebo>
+    <!-- simulate a body pose sensor -->
+    <gazebo>
+        <plugin name="p3d" filename="libgazebo_ros_p3d.so">
+        <alwaysOn>true</alwaysOn>
+        <updateRate>100.0</updateRate>
+        <bodyName>base</bodyName>
+        <topicName>body_pose_ground_truth</topicName>
+        <frameName>world</frameName>
+        <xyzOffsets>0 0 0.0</xyzOffsets>
+        <rpyOffsets>0 0 0.0</rpyOffsets>
+        </plugin>
+    </gazebo>
+    <gazebo>
+        <plugin name="p3d" filename="libgazebo_ros_p3d.so">
+            <always_on>true</always_on>
+            <update_rate>200</update_rate>
+            <bodyName>base</bodyName>
+            <topicName>/torso_odom</topicName>
+            <frameName>world</frameName>
+            <xyzOffset>0 0 0</xyzOffset>
+            <rpyOffset>0 0 0</rpyOffset>
+        </plugin>
+    </gazebo>
     <!-- Show the trajectory of trunk center. -->
-    <gazebo>
-        <plugin name="3dplot" filename="libLinkPlot3DPlugin.so">
-            <frequency>10</frequency>
-            <plot>
-                <link>base</link>
-                <pose>0 0 0 0 0 0</pose>
-                <material>Gazebo/Yellow</material>
-            </plot>
-        </plugin>
-    </gazebo>
-    <!-- Show the trajectory of foot. You can add another trajectory about another foot. -->
-    <!-- <gazebo>
-        <plugin name="3dplot" filename="libLinkPlot3DPlugin.so">
-            <frequency>100</frequency>
-            <plot>
-                <link>FL_foot</link>
-                <pose>0 0 0 0 0 0</pose>
-                <material>Gazebo/Green</material>
-            </plot>
-        </plugin>
-    </gazebo> -->
     <gazebo>
         <plugin filename="libgazebo_ros_force.so" name="gazebo_ros_force">
@@ -40,5 +42,5 @@
         <sensor name="imu_sensor" type="imu">
             <always_on>true</always_on>
-            <update_rate>1000</update_rate>
+            <update_rate>400</update_rate>
             <visualize>true</visualize>
             <topic>__default_topic__</topic>
@@ -46,6 +48,6 @@
                 <topicName>trunk_imu</topicName>
                 <bodyName>imu_link</bodyName>
-                <updateRateHZ>1000.0</updateRateHZ>
-                <gaussianNoise>0.0</gaussianNoise>
+                <updateRateHZ>400.0</updateRateHZ>
+                <gaussianNoise>0.001</gaussianNoise>
                 <xyzOffset>0 0 0</xyzOffset>
                 <rpyOffset>0 0 0</rpyOffset>

File: robots/a1_description/xacro/robot.xacro (robot description, xacro)
@@ -6,5 +6,4 @@
     <xacro:include filename="$(find a1_description)/xacro/stairs.xacro"/>
     <xacro:include filename="$(find a1_description)/xacro/gazebo.xacro"/>
-    <!-- <xacro:include filename="$(find a1_gazebo)/launch/stairs.urdf.xacro"/> -->
     <!-- <xacro:stairs stairs="15" xpos="0" ypos="0" zpos="0" /> -->
     <!-- Rollover Protection mode will add an additional stick on the top, use "true" or "false" to switch it. -->
@@ -43,5 +42,5 @@
             <origin rpy="0 0 0" xyz="0 0 0"/>
             <geometry>
-                <box size="${trunk_length} ${trunk_width} ${trunk_height}"/>
+                <mesh filename="package://a1_description/meshes/trunk.dae" scale="1 1 1"/>
             </geometry>
         </collision>
