Commit message: fix go1 gazebo bug

File: robots/go1_description/xacro/robot.xacro (robot description, xacro)
@@ -4,10 +4,7 @@
     <xacro:include filename="$(find go1_description)/xacro/materials.xacro"/>
     <xacro:include filename="$(find go1_description)/xacro/leg.xacro"/>
-    <!-- <xacro:include filename="$(find go1_description)/xacro/stairs.xacro"/> -->
     <xacro:include filename="$(find go1_description)/xacro/gazebo.xacro"/>
     <xacro:include filename="$(find go1_description)/xacro/depthCamera.xacro"/>
     <xacro:include filename="$(find go1_description)/xacro/ultraSound.xacro"/>
-    <!-- <xacro:include filename="$(find go1_gazebo)/launch/stairs.urdf.xacro"/> -->
-    <!-- <xacro:stairs stairs="15" xpos="0" ypos="0" zpos="0" /> -->
     <!-- Rollover Protection mode will add an additional stick on the top, use "true" or "false" to switch it. -->
     <xacro:property name="rolloverProtection" value="false"/>
@@ -40,5 +37,4 @@
                 <mesh filename="package://go1_description/meshes/trunk.dae" scale="1 1 1"/>
             </geometry>
-            <!-- <material name="orange"/> -->
         </visual>
         <collision>
@@ -69,5 +65,4 @@
                 </geometry>
                 <origin rpy="0 0 0" xyz="0 0 0"/>
-                <!-- <material name="white"/> -->
             </visual>
             <collision>
@@ -102,5 +97,4 @@
                 <box size="0.001 0.001 0.001"/>
             </geometry>
-            <!-- <material name="red"/> -->
         </visual>
         <collision>
